Commit message: wfe

File: tt_env/envs/robot/robot.urdf (robot description, URDF)
Before this commit: robot onshape, 5 links, 4 joints
Links:
- removed link link_l0
- removed link link_l1
- removed link link_l2
- removed link link_l3
- removed link link_l4
- added link l0, mass 31.011862534247164547; collision mesh filename=package:///l0.stl; visual mesh filename=package:///l0.stl
- added link l1, mass 13.447711806464676343; collision mesh filename=package:///l1.stl; visual mesh filename=package:///l1.stl
- added link l2, mass 3.3373406335618427399; collision mesh filename=package:///l2.stl; visual mesh filename=package:///l2.stl
- added link l3, mass 4.3185906335617918472; collision mesh filename=package:///l3.stl; visual mesh filename=package:///l3.stl
- added link l4, mass 1.3020665219465743512; collision mesh filename=package:///l4.stl; visual mesh filename=package:///l4.stl
- added link l5, mass 2.8350584440449333457; collision mesh filename=package:///l5.stl; visual mesh filename=package:///l5.stl
Joints:
- added joint j4_continuous: type revolute, parent l4, child l5, origin xyz=-2.1807555761199637345e-11 -0.10249233999943557771 -0.0010000000000001119105 rpy=1.5707963267948974462 -1.4415324059003871149 3.1415926535897611416, axis 0 0 1, limit effort=1 velocity=20
- joint j0_continuous: child link_l1 -> l1; origin xyz=-5.5511151231257827021e-17 -1.7130394325270970057e-17 0.020000000000000000416 rpy=3.141592653589793116 -3.9064654370572275462e-20 -3.1372106767731211541 -> xyz=4.4433313139149082721e-20 -2.9354910603076127659e-18 0.10000000000000001943 rpy=-3.141592653589793116 1.0118004717258600843e-18 -0.0024120916050152920937; parent link_l0 -> l0
- joint j1: child link_l2 -> l2; limit lower=0 upper=3.8048177693476383787 effort=1 velocity=20 -> lower=1.0471975511965976313 upper=5.2359877559829888227 effort=1 velocity=20; origin xyz=0.019999999999999899802 0.013999999999999899677 -0.076000000000000109135 rpy=1.57079632679489678 -0.66322511575784137694 -3.141592653589793116 -> xyz=3.4208452816061431113e-16 -0.012499999999999997224 -0.10250000000000034084 rpy=1.57079632679489678 -0.65183928279709479892 -1.7774619825444202965e-15; parent link_l1 -> l1
- joint j2: child link_l3 -> l3; limit lower=0.087266462599716473902 upper=4.6251225177849732972 effort=1 velocity=20 -> effort=1 velocity=20; origin xyz=0.052873043309672435042 -0.066554047894725548717 -0.0049999999999999957673 rpy=1.3523355692128363387e-16 1.3845705657597024673e-14 -0.3831718014110614412 -> xyz=-1.9428902930940239457e-16 -0.35000000000000330846 -0.025000000000000015266 rpy=-3.1415926535897904515 3.4189179422415795443e-16 1.9872695389451910941; parent link_l2 -> l2
- joint j3_continuous: child link_l4 -> l4; origin xyz=0.0031672005010480244747 0.02379009964220740736 -0.0089999999999999923811 rpy=1.5707963267948994446 1.5701450367702478594 -0.13235275869594265163 -> xyz=-5.5511151231257827021e-17 0.45000000000000006661 -0.012500000000000004163 rpy=-1.570796326794896558 1.5440601655300412176 3.1415926535897193972; parent link_l3 -> l3

File: tt_env/envs/table/robot.urdf (robot description, URDF)
Before this commit: robot onshape, 1 links, 0 joints
Links:
- link table: mass 0.5408016000000003265 -> 66.930420000000026448
